File: hardware/main_controller_hat/Project Architecture.kicad_sch (KiCad schematic)
At the start: 4 parts

Commit message: revise main controller with pc817
Parts:
- renumbered H2 to H1, H1 to H2
Changed lines of the file:
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@@
 		(dnp no)
 		(fields_autoplaced yes)
-		(property "Reference" "H1"
+		(property "Reference" "H2"
 			(at 256.54 104.1399 0)
 			(show_name no)
@@
 			(project "main_controller_hat"
 				(path "/f9e05184-c88b-4a88-ae9c-ab2bdb32be7c/c5103ceb-5325-4a84-a025-9638a412984e"
-					(reference "H1")
+					(reference "H2")
 					(unit 1)
 				)
@@
 		(dnp no)
 		(fields_autoplaced yes)
-		(property "Reference" "H2"
+		(property "Reference" "H1"
 			(at 255.27 114.2999 0)
 			(show_name no)
@@
 			(project "main_controller_hat"
 				(path "/f9e05184-c88b-4a88-ae9c-ab2bdb32be7c/c5103ceb-5325-4a84-a025-9638a412984e"
-					(reference "H2")
+					(reference "H1")
 					(unit 1)
 				)
