File: hardware/main_controller_hat/main_controller_hat.kicad_pcb (KiCad board)
At the start: 6 copper layers, 160 x 100 mm, 87 parts, among them J1 21V Li ion, J14 Screw_Terminal_01x06, J2 Conn_01x10_Pin, J3 RJ45_Hanrun_HR911105A_Horizon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, J4 CAN 1, J5 Conn_01x04_Pin, J6 UART, J7 ENC A, J8 ENC B, J9 CMPS14, Q1 IRFR5305, Q2 IRFR5305, Q3 BSS138, Q4 BSS138, Q5 BSS138, Q6 BSS138, U1 LM2596S-5, U10 6N137, U11 6N137, U12 BTS7960B, U13 BTS7960B, U14 LM2596S-5, U15 SN65HVD230, U3 AMS1117-3.3, U5 Teensy4.1, U6 6N137, U7 6N137, U8 BTS7960B, U9 BTS7960B

Commit message: main controller final design
Parts:
- C11, C2: footprint Capacitor_SMD:C_0603_1608Metric -> Capacitor_SMD:C_0805_2012Metric
- C13: footprint Capacitor_SMD:C_1206_3216Metric_Pad1.33x1.80mm_HandSolder -> Capacitor_SMD:C_0805_2012Metric
- C4, C6: footprint Capacitor_SMD:C_1206_3216Metric_Pad1.33x1.80mm_HandSolder -> Capacitor_SMD:C_1206_3216Metric
- C5, C7: footprint Capacitor_SMD:C_0603_1608Metric_Pad1.08x0.95mm_HandSolder -> Capacitor_SMD:C_0805_2012Metric
- R17, R18, R19: footprint Resistor_SMD:R_0603_1608Metric_Pad0.98x0.95mm_HandSolder -> Resistor_SMD:R_0805_2012Metric
Routing:
- net GND: track 235.9 -> 167.3 mm, vias 10 -> 28
- net R+: track 147.6 -> 146.3 mm
- net T-: track 143.0 -> 142.3 mm
- net +5V: track 304.9 -> 305.5 mm
- net T+: track 147.1 -> 146.5 mm
Other:
- board text added: "13"
- board text added: "33"
- board text added: "34"
- board text added: "35"
- board text added: "36"
- board text added: "37"
- board text added: "38"
- board text added: "39"
- board text added: "40"
- board text added: "41"
- board text added: "Ananta Pamungkas"
- board text added: "Main controller Autonomous Wheelchair v1.0 2026-08-13 Intelligent System and Robotics lab UNEJ"
- board text added: "TEENSY 4.1"

Commit message: revise main controller with pc817
Parts:
- removed the R10 at (157.5, 94.5)
- removed the R9 at (157.8, 62.8)
- removed the U11 at (153.8, 98.3)
- removed the U7 at (154.1, 82.6)
- added ?: , , F.Cu at (220.4, 41.5)
- added ?: , , F.Cu at (220.4, 39.5)
- added ?: , , F.Cu at (222.4, 39.5)
- added ?: , , F.Cu at (220.4, 37.5)
- added ?: , , F.Cu at (222.4, 41.5)
- added ?: , , F.Cu at (222.4, 37.5)
- added J7: RJ45_Hanrun_HR911105A_Horizontal, Connector_RJ:RJ45_Hanrun_HR911105A_Horizontal, F.Cu at (213.9, 38.1)
- added R14: 220, Resistor_SMD:R_0805_2012Metric, F.Cu at (161.1, 69.0)
- added R15: 220, Resistor_SMD:R_0805_2012Metric, F.Cu at (161.0, 76.0)
- added R16: 220, Resistor_SMD:R_0805_2012Metric, F.Cu at (145.0, 69.0)
- added R17: 220, Resistor_SMD:R_0805_2012Metric, F.Cu at (145.0, 76.0)
- added R5: 220, Resistor_SMD:R_0805_2012Metric, F.Cu at (161.0, 62.0)
- added R6: 220, Resistor_SMD:R_0805_2012Metric, F.Cu at (145.0, 83.0)
- added R7: 220, Resistor_SMD:R_0805_2012Metric, F.Cu at (145.0, 55.0)
- added R8: 220, Resistor_SMD:R_0805_2012Metric, F.Cu at (145.0, 62.0)
- added U4: PC817X2NIP1B, PC817X2NIP1B:SOIC254P960X420-4N, F.Cu at (153.0, 83.0)
- added U5: PC817X2NIP1B, PC817X2NIP1B:SOIC254P960X420-4N, F.Cu at (153.0, 55.0)
- added U9: PC817X2NIP1B, PC817X2NIP1B:SOIC254P960X420-4N, F.Cu at (153.0, 69.0)
- D10: renamed from D9; footprint PCM_SparkFun-LED:LED_0805_2012Metric -> LED_SMD:LED_0805_2012Metric
- D5: footprint PCM_SparkFun-LED:LED_0805_2012Metric -> LED_SMD:LED_0805_2012Metric
- J3: value RJ45_Hanrun_HR911105A_Horizontal -> EN; footprint Connector_RJ:RJ45_Hanrun_HR911105A_Horizontal -> Connector_PinSocket_2.54mm:PinSocket_1x02_P2.54mm_Vertical
- R1: renamed from R2; footprint PCM_SparkFun-Resistor:R_0805_2012Metric -> Resistor_SMD:R_0805_2012Metric
- R10: renamed from R13; footprint PCM_SparkFun-Resistor:R_0805_2012Metric -> Resistor_SMD:R_0805_2012Metric
- R11: renamed from R16; footprint PCM_SparkFun-Resistor:R_0805_2012Metric -> Resistor_SMD:R_0805_2012Metric
- R12: renamed from R5; footprint PCM_SparkFun-Resistor:R_0805_2012Metric -> Resistor_SMD:R_0805_2012Metric
- R13: renamed from R11; footprint PCM_SparkFun-Resistor:R_0805_2012Metric -> Resistor_SMD:R_0805_2012Metric
- R18: renamed from R8; footprint PCM_SparkFun-Resistor:R_0805_2012Metric -> Resistor_SMD:R_0805_2012Metric
- R19: renamed from R14; footprint PCM_SparkFun-Resistor:R_0805_2012Metric -> Resistor_SMD:R_0805_2012Metric
- R2: renamed from R1; footprint PCM_SparkFun-Resistor:R_0805_2012Metric -> Resistor_SMD:R_0805_2012Metric
- R20: renamed from R6; footprint PCM_SparkFun-Resistor:R_0805_2012Metric -> Resistor_SMD:R_0805_2012Metric
- R21: renamed from R12; footprint PCM_SparkFun-Resistor:R_0805_2012Metric -> Resistor_SMD:R_0805_2012Metric
- R22: renamed from R15; footprint PCM_SparkFun-Resistor:R_0805_2012Metric -> Resistor_SMD:R_0805_2012Metric
- R26: renamed from R20; footprint PCM_SparkFun-Resistor:R_0805_2012Metric -> Resistor_SMD:R_0805_2012Metric
- R27: renamed from R24; footprint PCM_SparkFun-Resistor:R_0805_2012Metric -> Resistor_SMD:R_0805_2012Metric
- R28: renamed from R21; footprint PCM_SparkFun-Resistor:R_0805_2012Metric -> Resistor_SMD:R_0805_2012Metric
- R29: renamed from R25; footprint PCM_SparkFun-Resistor:R_0805_2012Metric -> Resistor_SMD:R_0805_2012Metric
- R3, R4: value 10K -> 220; footprint PCM_SparkFun-Resistor:R_0805_2012Metric -> Resistor_SMD:R_0805_2012Metric; moved to F.Cu
- R30: renamed from R22; footprint PCM_SparkFun-Resistor:R_0805_2012Metric -> Resistor_SMD:R_0805_2012Metric
- R31: renamed from R26; footprint PCM_SparkFun-Resistor:R_0805_2012Metric -> Resistor_SMD:R_0805_2012Metric
- R32: renamed from R23; footprint PCM_SparkFun-Resistor:R_0805_2012Metric -> Resistor_SMD:R_0805_2012Metric
- R33: renamed from R27; footprint PCM_SparkFun-Resistor:R_0805_2012Metric -> Resistor_SMD:R_0805_2012Metric
- R9: renamed from R7; footprint PCM_SparkFun-Resistor:R_0805_2012Metric -> Resistor_SMD:R_0805_2012Metric
- U10, U6: value 6N137 -> PC817X2NIP1B; footprint Package_DIP:DIP-8_W7.62mm -> PC817X2NIP1B:SOIC254P960X420-4N
- moved J3 91.4 mm to (148.6, 94.2)
- moved R3 36.4 mm to (161.0, 83.0), turned to -90 degrees
- moved R4 24.0 mm to (161.0, 55.0), turned to -90 degrees
- moved R25 17.9 mm to (220.7, 27.7), turned to -90 degrees
- moved U6 11.5 mm to (153.0, 62.0)
- moved U10 9.49 mm to (153.0, 76.0)
- moved C12 6.29 mm to (207.8, 34.8), turned to 0 degrees
- renumbered C4 to C1, C11 to C10, C12 to C11, C13 to C12, C5 to C2, C6 to C3, C7 to C4, C1 to C5, C2 to C6, C3 to C7, C10 to C9, D3 to D1, D1 to D2, D4 to D3, D2 to D4, D10 to D6, D6 to D9, H2 to H1, H1 to H2, J7 to J10, J8 to J11, J14 to J4, J4 to J5, J5 to J6, J6 to J8, Q5 to Q4, Q4 to Q5, R19 to R23, R17 to R24, R18 to R25, U3 to U1, U9 to U11, U13 to U12, U14 to U13, U15 to U14, U1 to U2, U5 to U3, U8 to U7, U12 to U8
Connections:
- C12 pad 2: Net-(J3-RCT) -> Net-(J7-RCT)
- J3 pad 1: T+ -> ENABLE_SIG
- J3 pad 2: T- -> +5VA
- R25 pad 1: Net-(J3-Pad9) -> Net-(J7-Pad9)
- R3 pad 1: RPWM -> ENABLE_PIN
- R3 pad 2: GND -> Net-(R3-Pad2)
- R4 pad 1: RPWM1 -> RPWM
- R4 pad 2: GND -> Net-(R4-Pad2)
- U10 pad 1: unconnected-(U10-NC-Pad1) -> Net-(R15-Pad2)
- U10 pad 2: LPWM -> GND
- U10 pad 3: GND -> Net-(U12-IN)
- U10 pad 4: unconnected-(U10-NC-Pad4) -> +5VA
- U11 pad 3: +5VA -> ENABLE_SIG
- U12 pad 2: Net-(U11-VO) -> Net-(U12-IN)
- U12 pad 3: +5VA -> ENABLE_SIG
- U3 pad 16: unconnected-(U5-24_A10_TX6_SCL2-Pad16) -> ENABLE_PIN
- U3 pad 34: unconnected-(U5-GND-Pad34) -> GND
- U3 pad 47: unconnected-(U5-GND-Pad47) -> GND
- U6 pad 1: unconnected-(U6-NC-Pad1) -> Net-(R5-Pad2)
- U6 pad 2: RPWM -> GND
- U6 pad 3: GND -> Net-(U8-IN)
- U6 pad 4: unconnected-(U6-NC-Pad4) -> +5VA
- U7 pad 2: Net-(U6-VO) -> Net-(U7-IN)
- U7 pad 3: +5VA -> ENABLE_SIG
- U8 pad 2: Net-(U10-VO) -> Net-(U8-IN)
- U8 pad 3: +5VA -> ENABLE_SIG
Routing:
- net R+: track 146.3 -> 10.5 mm, vias 2 -> 0
- net T-: track 142.3 -> 7.53 mm, vias 3 -> 0
- net T+: track 146.5 -> 13.8 mm, vias 2 -> 0
- net R-: track 149.9 -> 26.2 mm, vias 2 -> 0
- net ENABLE_PIN: track 0.00 -> 100.2 mm, vias 0 -> 2
- net +5VA: track 207.4 -> 128.6 mm
- net ENABLE_SIG: track 0.00 -> 73.6 mm, vias 0 -> 4
- net GND: track 167.3 -> 94.5 mm, vias 28 -> 37
- net +3.3V: track 340.8 -> 398.7 mm, vias 7 -> 5
- net GNDA: track 70.0 -> 114.1 mm, vias 13 -> 20
- net Net-(U12-IN): track 0.00 -> 31.6 mm
- net LPWM1: track 123.5 -> 100.9 mm, vias 0 -> 1
- net Net-(U7-IN): track 0.00 -> 18.2 mm
- net LED: track 42.6 -> 27.1 mm
- net unconnected-(J7-PadSH): track 0.00 -> 15.5 mm
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- added copper zone on B.Cu, net ENABLE_SIG
Other:
- board text added: "ENABLE"
- board text added: "Ethernet"
- board text added: "Main controller Autonomous Wheelchair v1.1 2026-08-10 Intelligent System and Robotics lab UNEJ"
- board text added: "RJ45"
- board text removed: "Ananta Pamungkas"
- board text removed: "Main controller Autonomous Wheelchair v1.0 2026-08-13 Intelligent System and Robotics lab UNEJ"
