File: hardware/main_controller_hat/motor_controller.kicad_sch (KiCad schematic)
At the start: 36 parts, among them J14 Screw_Terminal_01x06, Q2 IRFR5305, U10 6N137, U11 6N137, U12 BTS7960B, U13 BTS7960B, U14 LM2596S-5, U6 6N137, U7 6N137, U8 BTS7960B, U9 BTS7960B

Commit message: main controller final design
Parts:
- C11: footprint Capacitor_SMD:C_0603_1608Metric -> Capacitor_SMD:C_0805_2012Metric

Commit message: revise main controller with pc817
Parts:
- removed R10, R9: 10K, PCM_SparkFun-Resistor:R_0805_2012Metric, symbol Device:R
- removed U10, U11, U6, U7: 6N137, Package_DIP:DIP-8_W7.62mm, symbol Isolator:6N137
- added J3: EN, Connector_PinSocket_2.54mm:PinSocket_1x02_P2.54mm_Vertical, symbol Connector:Conn_01x02_Pin
- added R14, R15, R16, R17, R5, R6, R7, R8: 220, Resistor_SMD:R_0805_2012Metric, symbol Device:R
- added U10, U4, U5, U6, U9: PC817X2NIP1B, PC817X2NIP1B:SOIC254P960X420-4N, symbol PC817X2NIP1B:PC817X2NIP1B
- D10: renamed from D9; footprint PCM_SparkFun-LED:LED_0805_2012Metric -> LED_SMD:LED_0805_2012Metric
- R10: renamed from R13; footprint PCM_SparkFun-Resistor:R_0805_2012Metric -> Resistor_SMD:R_0805_2012Metric
- R11: renamed from R16; footprint PCM_SparkFun-Resistor:R_0805_2012Metric -> Resistor_SMD:R_0805_2012Metric
- R12: renamed from R5; footprint PCM_SparkFun-Resistor:R_0805_2012Metric -> Resistor_SMD:R_0805_2012Metric
- R13: renamed from R11; footprint PCM_SparkFun-Resistor:R_0805_2012Metric -> Resistor_SMD:R_0805_2012Metric
- R18: renamed from R8; footprint PCM_SparkFun-Resistor:R_0805_2012Metric -> Resistor_SMD:R_0805_2012Metric
- R19: renamed from R14; footprint PCM_SparkFun-Resistor:R_0805_2012Metric -> Resistor_SMD:R_0805_2012Metric
- R20: renamed from R6; footprint PCM_SparkFun-Resistor:R_0805_2012Metric -> Resistor_SMD:R_0805_2012Metric
- R21: renamed from R12; footprint PCM_SparkFun-Resistor:R_0805_2012Metric -> Resistor_SMD:R_0805_2012Metric
- R22: renamed from R15; footprint PCM_SparkFun-Resistor:R_0805_2012Metric -> Resistor_SMD:R_0805_2012Metric
- R3, R4: value 10K -> 220; footprint PCM_SparkFun-Resistor:R_0805_2012Metric -> Resistor_SMD:R_0805_2012Metric
- R9: renamed from R7; footprint PCM_SparkFun-Resistor:R_0805_2012Metric -> Resistor_SMD:R_0805_2012Metric
- renumbered C11 to C10, C12 to C11, C10 to C9, D10 to D6, D6 to D9, J14 to J4, U9 to U11, U13 to U12, U14 to U13, U8 to U7, U12 to U8
Connections:
- net +5VA: now also J3.2 (Pin_2), U10.4, U4.4, U5.4, U6.4, U9.4; no longer U11.3 (INH), U12.3 (INH), U7.3 (INH), U8.3 (INH)
- net GND: now also U10.2, U4.2, U5.2, U6.2, U9.2; no longer R3.2, R4.2
- net GNDA: now also R16.1, R17.1, R6.1, R7.1, R8.1
- net LPWM: now also R5.1
- net LPWM1: now also R15.1
- net RPWM: now also R4.1; no longer R3.1
- net RPWM1: now also R14.1; no longer R4.1
- net at U12.2 (IN): now also R17.2, U10.3
- net at U8.2 (IN): now also R8.2, U6.3
- net at U11.2 (IN): now also R16.2, U9.3
- net at U7.2 (IN): now also R7.2, U5.3
- new net: R5.2, U6.1
- new net: R15.2, U10.1
- new net: R4.2, U5.1
- new net: R3.2, U4.1
- new net: R14.2, U9.1
- new net ENABLE_PIN: R3.1
- new net ENABLE_SIG: J3.1 (Pin_1), R6.2, U11.3 (INH), U12.3 (INH), U4.3, U7.3 (INH), U8.3 (INH)
Other:
- moved on the sheet: C8, D6, D7, FH2, J4, Q2, R10, R11, R12, R13, R18, R19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
