File: hardware/main_controller_hat/sensor.kicad_sch (KiCad schematic)
At the start: 15 parts, among them J7 ENC A, J8 ENC B, J9 CMPS14, Q3 BSS138, Q4 BSS138, Q5 BSS138, Q6 BSS138

Commit message: revise main controller with pc817
Parts:
- R26: renamed from R20; footprint PCM_SparkFun-Resistor:R_0805_2012Metric -> Resistor_SMD:R_0805_2012Metric
- R27: renamed from R24; footprint PCM_SparkFun-Resistor:R_0805_2012Metric -> Resistor_SMD:R_0805_2012Metric
- R28: renamed from R21; footprint PCM_SparkFun-Resistor:R_0805_2012Metric -> Resistor_SMD:R_0805_2012Metric
- R29: renamed from R25; footprint PCM_SparkFun-Resistor:R_0805_2012Metric -> Resistor_SMD:R_0805_2012Metric
- R30: renamed from R22; footprint PCM_SparkFun-Resistor:R_0805_2012Metric -> Resistor_SMD:R_0805_2012Metric
- R31: renamed from R26; footprint PCM_SparkFun-Resistor:R_0805_2012Metric -> Resistor_SMD:R_0805_2012Metric
- R32: renamed from R23; footprint PCM_SparkFun-Resistor:R_0805_2012Metric -> Resistor_SMD:R_0805_2012Metric
- R33: renamed from R27; footprint PCM_SparkFun-Resistor:R_0805_2012Metric -> Resistor_SMD:R_0805_2012Metric
- renumbered J7 to J10, J8 to J11, Q5 to Q4, Q4 to Q5
